File: src/interface.sch (KiCad schematic (older format))
At the start: 8 parts

Commit message: Substituição dos transitores NMOS pelo transistor 2n7000
Parts:
- Q? (x2): value Q_NMOS_DGS -> 2n7000
Changed lines of the file:
@@
 P 4350 1950
 F 0 "Q?" H 4650 2000 50  0000 R CNN
-F 1 "Q_NMOS_DGS" H 5000 1900 50  0000 R CNN
+F 1 "2n7000" H 5000 1900 50  0000 R CNN
 F 2 "" H 4550 2050 50  0000 C CNN
 F 3 "" H 4350 1950 50  0000 C CNN
@@
 P 5950 3200
 F 0 "Q?" H 6250 3250 50  0000 R CNN
-F 1 "Q_NMOS_DGS" H 6600 3150 50  0000 R CNN
+F 1 "2n7000" H 6600 3150 50  0000 R CNN
 F 2 "" H 6150 3300 50  0000 C CNN
 F 3 "" H 5950 3200 50  0000 C CNN

Commit message: Verificação ERC -- checagem de erros elétricos no esquema -- concluída com sucesso. Há apenas dois warnings que não indicam problemas.
Parts:
- gave numbers to parts that had none: 8
Changed lines of the file:
@@
 _REQUEST_UNLOCK
 $Comp
-L +3.3V #PWR?
+L +3.3V #PWR021
 U 1 1 57CDF4C9
 P 4450 1450
-F 0 "#PWR?" H 4450 1300 50  0001 C CNN
+F 0 "#PWR021" H 4450 1300 50  0001 C CNN
 F 1 "+3.3V" H 4450 1590 50  0000 C CNN
 F 2 "" H 4450 1450 50  0000 C CNN
@@
 $EndComp
 $Comp
-L GND #PWR?
+L GND #PWR022
 U 1 1 57CDF4DD
 P 4450 3100
-F 0 "#PWR?" H 4450 2850 50  0001 C CNN
+F 0 "#PWR022" H 4450 2850 50  0001 C CNN
 F 1 "GND" H 4450 2950 50  0000 C CNN
 F 2 "" H 4450 3100 50  0000 C CNN
@@
 $EndComp
 $Comp
-L Q_NMOS_DGS Q?
+L Q_NMOS_DGS Q1
 U 1 1 57CDF55A
 P 4350 1950
-F 0 "Q?" H 4650 2000 50  0000 R CNN
+F 0 "Q1" H 4650 2000 50  0000 R CNN
 F 1 "2n7000" H 5000 1900 50  0000 R CNN
 F 2 "" H 4550 2050 50  0000 C CNN
@@
 $EndComp
 $Comp
-L Q_NMOS_DGS Q?
+L Q_NMOS_DGS Q2
 U 1 1 57CDF617
 P 5950 3200
-F 0 "Q?" H 6250 3250 50  0000 R CNN
+F 0 "Q2" H 6250 3250 50  0000 R CNN
 F 1 "2n7000" H 6600 3150 50  0000 R CNN
 F 2 "" H 6150 3300 50  0000 C CNN
@@
 $EndComp
 $Comp
-L GND #PWR?
+L GND #PWR023
 U 1 1 57CDF79A
 P 6050 3650
-F 0 "#PWR?" H 6050 3400 50  0001 C CNN
+F 0 "#PWR023" H 6050 3400 50  0001 C CNN
 F 1 "GND" H 6050 3500 50  0000 C CNN
 F 2 "" H 6050 3650 50  0000 C CNN
@@
 $EndComp
 $Comp
-L +3.3V #PWR?
+L +3.3V #PWR024
 U 1 1 57CDF7CB
 P 6050 2350
-F 0 "#PWR?" H 6050 2200 50  0001 C CNN
+F 0 "#PWR024" H 6050 2200 50  0001 C CNN
 F 1 "+3.3V" H 6050 2490 50  0000 C CNN
 F 2 "" H 6050 2350 50  0000 C CNN
@@
 $EndComp
 $Comp
-L LED D?
+L LED D3
 U 1 1 57CDF7DC
 P 4450 2850
-F 0 "D?" H 4450 2950 50  0000 C CNN
+F 0 "D3" H 4450 2950 50  0000 C CNN
 F 1 "LED VERDE" H 4450 2750 50  0000 C CNN
 F 2 "" H 4450 2850 50  0000 C CNN
@@
 $EndComp
 $Comp
-L LED D?
+L LED D4
 U 1 1 57CDF888
 P 6750 3150
-F 0 "D?" H 6750 3250 50  0000 C CNN
+F 0 "D4" H 6750 3250 50  0000 C CNN
 F 1 "LED VERMELHO" H 6750 3050 50  0000 C CNN
 F 2 "" H 6750 3150 50  0000 C CNN
@@
 $EndComp
 $Comp
-L R R?
+L R R31
 U 1 1 57CDF9A0
 P 4450 2450
-F 0 "R?" V 4530 2450 50  0000 C CNN
+F 0 "R31" V 4530 2450 50  0000 C CNN
 F 1 "150" V 4450 2450 50  0000 C CNN
 F 2 "" V 4380 2450 50  0000 C CNN
@@
 $EndComp
 $Comp
-L R R?
+L R R32
 U 1 1 57CDFA48
 P 6050 2650
-F 0 "R?" V 6130 2650 50  0000 C CNN
+F 0 "R32" V 6130 2650 50  0000 C CNN
 F 1 "220" V 6050 2650 50  0000 C CNN
 F 2 "" V 5980 2650 50  0000 C CNN
@@
 Connection ~ 3900 1950
 $Comp
-L SPST SW?
+L SPST SW1
 U 1 1 57CE08F4
 P 7850 2350
-F 0 "SW?" H 7850 2450 50  0000 C CNN
+F 0 "SW1" H 7850 2450 50  0000 C CNN
 F 1 "SPST" H 7850 2250 50  0000 C CNN
 F 2 "" H 7850 2350 50  0000 C CNN
@@
 $EndComp
 $Comp
-L GND #PWR?
+L GND #PWR025
 U 1 1 57CE09A9
 P 7300 2500
-F 0 "#PWR?" H 7300 2250 50  0001 C CNN
+F 0 "#PWR025" H 7300 2250 50  0001 C CNN
 F 1 "GND" H 7300 2350 50  0000 C CNN
 F 2 "" H 7300 2500 50  0000 C CNN
@@
 $EndComp
 $Comp
-L R R?
+L R R33
 U 1 1 57CE0ACF
 P 8500 2000
-F 0 "R?" V 8580 2000 50  0000 C CNN
+F 0 "R33" V 8580 2000 50  0000 C CNN
 F 1 "220" V 8500 2000 50  0000 C CNN
 F 2 "" V 8430 2000 50  0000 C CNN
@@
 Connection ~ 8500 2350
 $Comp
-L +3.3V #PWR?
+L +3.3V #PWR026
 U 1 1 57CE0D74
 P 8500 1650
-F 0 "#PWR?" H 8500 1500 50  0001 C CNN
+F 0 "#PWR026" H 8500 1500 50  0001 C CNN
 F 1 "+3.3V" H 8500 1790 50  0000 C CNN
 F 2 "" H 8500 1650 50  0000 C CNN

Commit message: Footprint atualizado
Parts:
- D3, D4: footprint (none) -> LEDs:LED-5MM
- Q1, Q2: footprint (none) -> TO_SOT_Packages_THT:TO-92_Inline_Narrow_Oval
- R31, R32, R33: footprint (none) -> Resistors_ThroughHole:Resistor_Horizontal_RM7mm
- SW1: footprint (none) -> Buttons_Switches_ThroughHole:SW_PUSH-12mm
Changed lines of the file:
@@
 F 0 "Q1" H 4650 2000 50  0000 R CNN
 F 1 "2n7000" H 5000 1900 50  0000 R CNN
-F 2 "" H 4550 2050 50  0000 C CNN
+F 2 "TO_SOT_Packages_THT:TO-92_Inline_Narrow_Oval" H 4550 2050 50  0001 C CNN
 F 3 "" H 4350 1950 50  0000 C CNN
 	1    4350 1950
@@
 F 0 "Q2" H 6250 3250 50  0000 R CNN
 F 1 "2n7000" H 6600 3150 50  0000 R CNN
-F 2 "" H 6150 3300 50  0000 C CNN
+F 2 "TO_SOT_Packages_THT:TO-92_Inline_Narrow_Oval" H 6150 3300 50  0001 C CNN
 F 3 "" H 5950 3200 50  0000 C CNN
 	1    5950 3200
@@
 F 0 "D3" H 4450 2950 50  0000 C CNN
 F 1 "LED VERDE" H 4450 2750 50  0000 C CNN
-F 2 "" H 4450 2850 50  0000 C CNN
+F 2 "LEDs:LED-5MM" H 4450 2850 50  0001 C CNN
 F 3 "" H 4450 2850 50  0000 C CNN
 	1    4450 2850
@@
 F 0 "D4" H 6750 3250 50  0000 C CNN
 F 1 "LED VERMELHO" H 6750 3050 50  0000 C CNN
-F 2 "" H 6750 3150 50  0000 C CNN
+F 2 "LEDs:LED-5MM" H 6750 3150 50  0001 C CNN
 F 3 "" H 6750 3150 50  0000 C CNN
 	1    6750 3150
@@
 F 0 "R31" V 4530 2450 50  0000 C CNN
 F 1 "150" V 4450 2450 50  0000 C CNN
-F 2 "" V 4380 2450 50  0000 C CNN
+F 2 "Resistors_ThroughHole:Resistor_Horizontal_RM7mm" V 4380 2450 50  0001 C CNN
 F 3 "" H 4450 2450 50  0000 C CNN
 	1    4450 2450
@@
 F 0 "R32" V 6130 2650 50  0000 C CNN
 F 1 "220" V 6050 2650 50  0000 C CNN
-F 2 "" V 5980 2650 50  0000 C CNN
+F 2 "Resistors_ThroughHole:Resistor_Horizontal_RM7mm" V 5980 2650 50  0001 C CNN
 F 3 "" H 6050 2650 50  0000 C CNN
 	1    6050 2650
@@
 F 0 "SW1" H 7850 2450 50  0000 C CNN
 F 1 "SPST" H 7850 2250 50  0000 C CNN
-F 2 "" H 7850 2350 50  0000 C CNN
+F 2 "Buttons_Switches_ThroughHole:SW_PUSH-12mm" H 7850 2350 50  0001 C CNN
 F 3 "" H 7850 2350 50  0000 C CNN
 	1    7850 2350
@@
 F 0 "R33" V 8580 2000 50  0000 C CNN
 F 1 "220" V 8500 2000 50  0000 C CNN
-F 2 "" V 8430 2000 50  0000 C CNN
+F 2 "Resistors_ThroughHole:Resistor_Horizontal_RM7mm" V 8430 2000 50  0001 C CNN
 F 3 "" H 8500 2000 50  0000 C CNN
 	1    8500 2000
