File: src/trava_v2.sch (KiCad schematic (older format))
At the start: 6 parts

Commit message: Verificação ERC -- checagem de erros elétricos no esquema -- concluída com sucesso. Há apenas dois warnings que não indicam problemas.
Parts:
- added R35, R36: 0R, symbol R
- gave numbers to parts that had none: 6
Connections:
- net at IC1.6 (2Y), R30.2: now also R36.1; no longer IC1.11 (3Y)
- net at IC1.3 (1Y), R29.2: now also R35.1; no longer IC1.14 (4Y)
- new net: IC1.11 (3Y), R36.2
- new net: IC1.14 (4Y), R35.2
Changed lines of the file:
@@
 $EndDescr
 $Comp
-L L293D IC?
+L L293D IC1
 U 1 1 57C99E29
 P 5100 2300
-F 0 "IC?" H 4700 3140 50  0000 L CNN
+F 0 "IC1" H 4700 3140 50  0000 L CNN
 F 1 "L293D" H 4700 1400 50  0000 L CNN
 F 2 "DIL16" H 5100 2300 50  0001 L CNN
@@
 $EndComp
 $Comp
-L GND #PWR?
+L GND #PWR014
 U 1 1 57C9A1F1
 P 6200 2300
-F 0 "#PWR?" H 6200 2050 50  0001 C CNN
+F 0 "#PWR014" H 6200 2050 50  0001 C CNN
 F 1 "GND" H 6200 2150 50  0000 C CNN
 F 2 "" H 6200 2300 50  0000 C CNN
@@
 $EndComp
 $Comp
-L GND #PWR?
+L GND #PWR015
 U 1 1 57C9A206
 P 4250 2250
-F 0 "#PWR?" H 4250 2000 50  0001 C CNN
+F 0 "#PWR015" H 4250 2000 50  0001 C CNN
 F 1 "GND" H 4250 2100 50  0000 C CNN
 F 2 "" H 4250 2250 50  0000 C CNN
@@
 _LOCKED
 $Comp
-L CONN_01X05 P?
+L CONN_01X05 P4
 U 1 1 57C9E556
 P 9800 3200
-F 0 "P?" H 9800 3500 50  0000 C CNN
+F 0 "P4" H 9800 3500 50  0000 C CNN
 F 1 "LOCK_CONNECTOR" V 9900 3200 50  0000 C CNN
 F 2 "" H 9800 3200 50  0000 C CNN
@@
 $EndComp
 $Comp
-L R R?
+L R R29
 U 1 1 57C9E9EB
 P 8350 3000
-F 0 "R?" V 8430 3000 50  0000 C CNN
+F 0 "R29" V 8430 3000 50  0000 C CNN
 F 1 "R" V 8350 3000 50  0000 C CNN
 F 2 "" V 8280 3000 50  0000 C CNN
@@
 $EndComp
 $Comp
-L R R?
+L R R30
 U 1 1 57C9EB23
 P 8350 3400
-F 0 "R?" V 8430 3400 50  0000 C CNN
+F 0 "R30" V 8430 3400 50  0000 C CNN
 F 1 "R" V 8350 3400 50  0000 C CNN
 F 2 "" V 8280 3400 50  0000 C CNN
@@
 $EndComp
 $Comp
-L GND #PWR?
+L GND #PWR016
 U 1 1 57C9EC7E
 P 8100 3200
-F 0 "#PWR?" H 8100 2950 50  0001 C CNN
+F 0 "#PWR016" H 8100 2950 50  0001 C CNN
 F 1 "GND" H 8100 3050 50  0000 C CNN
 F 2 "" H 8100 3200 50  0000 C CNN
@@
 Text HLabel 2300 1950 0    60   Input ~ 0
 DIRECTION_L
-Wire Wire Line
-	4250 2200 4500 2200
-Wire Wire Line
-	4250 2200 4250 2250
-Wire Wire Line
-	4500 2400 4400 2400
-Wire Wire Line
-	4400 2400 4400 2200
-Connection ~ 4400 2200
-Wire Wire Line
-	6200 2200 6200 2300
-Wire Wire Line
-	5700 2200 6200 2200
-Wire Wire Line
-	5700 2400 5850 2400
-Wire Wire Line
-	5850 2400 5850 2200
-Connection ~ 5850 2200
-Wire Wire Line
-	2300 1800 4500 1800
-Wire Wire Line
-	5700 1800 6100 1800
-Wire Wire Line
-	6100 1800 6100 1200
-Wire Wire Line
-	6100 1200 4300 1200
-Wire Wire Line
-	4300 1200 4300 1800
-Connection ~ 4300 1800
-Wire Wire Line
-	4100 2000 4500 2000
-Wire Wire Line
-	4100 2000 4100 1050
-Wire Wire Line
-	4100 1050 6350 1050
-Wire Wire Line
-	6350 1050 6350 2000
-Wire Wire Line
-	5700 2000 7850 2000
-Connection ~ 6350 2000
-Wire Wire Line
-	4100 2600 4500 2600
-Wire Wire Line
-	5700 2600 7650 2600
-Wire Wire Line
-	7850 3000 8200 3000
-Wire Wire Line
-	8500 3000 9600 3000
-Wire Wire Line
-	8500 3400 9600 3400
-Wire Wire Line
-	7650 3400 8200 3400
-Wire Wire Line
-	8100 3200 9600 3200
-Wire Wire Line
-	8700 3100 9600 3100
-Wire Wire Line
-	8700 3750 8700 3100
-Wire Wire Line
-	7750 3750 8700 3750
-Wire Wire Line
-	8750 3300 9600 3300
-Wire Wire Line
-	8750 4000 8750 3300
-Wire Wire Line
-	7750 4000 8750 4000
-Wire Wire Line
-	3000 2800 4500 2800
-Wire Wire Line
-	4350 2800 4350 3300
-Wire Wire Line
-	4350 3300 5900 3300
-Wire Wire Line
-	5900 3300 5900 2800
-Wire Wire Line
-	5900 2800 5700 2800
-Wire Wire Line
-	6400 2600 6400 3800
-Wire Wire Line
-	6400 3800 4100 3800
-Wire Wire Line
-	4100 3800 4100 2600
-Connection ~ 6400 2600
-Wire Wire Line
-	3000 2800 3000 1950
-Wire Wire Line
-	3000 1950 2300 1950
-Connection ~ 4350 2800
-Wire Wire Line
-	7850 2000 7850 3000
-Wire Wire Line
-	7650 2600 7650 3400
-Wire Wire Line
-	2300 2150 2750 2150
-Wire Wire Line
-	2750 1600 2750 3500
-Wire Wire Line
-	2750 1600 4500 1600
-Wire Wire Line
-	5700 3500 5700 3000
-Wire Wire Line
-	2750 3500 5700 3500
-Connection ~ 2750 2150
-$Comp
-L +5V #PWR?
+$Comp
+L +5V #PWR017
 U 1 1 57C9F2D7
 P 6900 1200
-F 0 "#PWR?" H 6900 1050 50  0001 C CNN
+F 0 "#PWR017" H 6900 1050 50  0001 C CNN
 F 1 "+5V" H 6900 1340 50  0000 C CNN
 F 2 "" H 6900 1200 50  0000 C CNN
@@
 $EndComp
 $Comp
-L +12V #PWR?
+L +12V #PWR018
 U 1 1 57C9F2F3
 P 3500 2150
-F 0 "#PWR?" H 3500 2000 50  0001 C CNN
+F 0 "#PWR018" H 3500 2000 50  0001 C CNN
 F 1 "+12V" H 3500 2290 50  0000 C CNN
 F 2 "" H 3500 2150 50  0000 C CNN
@@
 	1    0    0    -1
 $EndComp
-Wire Wire Line
-	3800 3000 4500 3000
-Wire Wire Line
-	3800 2200 3800 3000
 Text Label 4250 2200 0    60   ~ 0
 NOTA1
 $Comp
-L GND #PWR?
+L GND #PWR019
 U 1 1 57C9F447
 P 6900 1750
-F 0 "#PWR?" H 6900 1500 50  0001 C CNN
+F 0 "#PWR019" H 6900 1500 50  0001 C CNN
 F 1 "GND" H 6900 1600 50  0000 C CNN
 F 2 "" H 6900 1750 50  0000 C CNN
@@
 $EndComp
 $Comp
-L C C?
+L C C5
 U 1 1 57C9F45C
 P 6900 1500
-F 0 "C?" H 6925 1600 50  0000 L CNN
+F 0 "C5" H 6925 1600 50  0000 L CNN
 F 1 "100nF" H 6925 1400 50  0000 L CNN
 F 2 "" H 6938 1350 50  0000 C CNN
@@
 	1    0    0    -1
 $EndComp
-Wire Wire Line
-	6900 1750 6900 1650
-Wire Wire Line
-	6900 1350 6900 1200
-Wire Wire Line
-	6900 1250 6500 1250
-Wire Wire Line
-	6500 1250 6500 1600
-Wire Wire Line
-	6500 1600 5700 1600
-Connection ~ 6900 1250
-$Comp
-L GND #PWR?
+$Comp
+L GND #PWR020
 U 1 1 57C9F6AD
 P 3500 2600
-F 0 "#PWR?" H 3500 2350 50  0001 C CNN
+F 0 "#PWR020" H 3500 2350 50  0001 C CNN
 F 1 "GND" H 3500 2450 50  0000 C CNN
 F 2 "" H 3500 2600 50  0000 C CNN
@@
 $EndComp
 $Comp
-L C C?
+L C C4
 U 1 1 57C9F72B
 P 3500 2400
-F 0 "C?" H 3525 2500 50  0000 L CNN
+F 0 "C4" H 3525 2500 50  0000 L CNN
 F 1 "100nF" H 3525 2300 50  0000 L CNN
 F 2 "" H 3538 2250 50  0000 C CNN
@@
 $EndComp
 Wire Wire Line
+	4250 2200 4500 2200
+Wire Wire Line
+	4250 2200 4250 2250
+Wire Wire Line
+	4500 2400 4400 2400
+Wire Wire Line
+	4400 2400 4400 2200
+Connection ~ 4400 2200
+Wire Wire Line
+	6200 2200 6200 2300
+Wire Wire Line
+	5700 2200 6200 2200
+Wire Wire Line
+	5700 2400 5850 2400
+Wire Wire Line
+	5850 2400 5850 2200
+Connection ~ 5850 2200
+Wire Wire Line
+	2300 1800 4500 1800
+Wire Wire Line
+	7850 3000 8200 3000
+Wire Wire Line
+	8500 3000 9600 3000
+Wire Wire Line
+	8500 3400 9600 3400
+Wire Wire Line
+	7650 3400 8200 3400
+Wire Wire Line
+	8100 3200 9600 3200
+Wire Wire Line
+	8700 3100 9600 3100
+Wire Wire Line
+	8700 3750 8700 3100
+Wire Wire Line
+	7750 3750 8700 3750
+Wire Wire Line
+	8750 3300 9600 3300
+Wire Wire Line
+	8750 4000 8750 3300
+Wire Wire Line
+	7750 4000 8750 4000
+Wire Wire Line
+	3000 2800 4500 2800
+Wire Wire Line
+	3000 2800 3000 1950
+Wire Wire Line
+	3000 1950 2300 1950
+Wire Wire Line
+	7850 2000 7850 3000
+Wire Wire Line
+	7650 2600 7650 3400
+Wire Wire Line
+	2300 2150 2750 2150
+Wire Wire Line
+	2750 1600 2750 3500
+Wire Wire Line
+	2750 1600 4500 1600
+Wire Wire Line
+	5700 3500 5700 3000
+Wire Wire Line
+	2750 3500 5700 3500
+Connection ~ 2750 2150
+Wire Wire Line
+	3800 3000 4500 3000
+Wire Wire Line
+	3800 2200 3800 3000
+Wire Wire Line
+	6900 1750 6900 1650
+Wire Wire Line
+	6900 1200 6900 1350
+Wire Wire Line
+	6900 1250 6500 1250
+Wire Wire Line
+	6500 1250 6500 1600
+Wire Wire Line
+	6500 1600 5700 1600
+Connection ~ 6900 1250
+Wire Wire Line
 	3800 2200 3500 2200
 Wire Wire Line
@@
 Wire Wire Line
 	3500 2550 3500 2600
+Wire Wire Line
+	5700 1800 5800 1800
+Wire Wire Line
+	5800 1800 5800 1300
+Wire Wire Line
+	5800 1300 4450 1300
+Wire Wire Line
+	4450 1300 4450 1800
+Connection ~ 4450 1800
+Wire Wire Line
+	4500 2000 4200 2000
+Wire Wire Line
+	4200 2000 4200 1100
+Wire Wire Line
+	4200 1100 6400 1100
+Wire Wire Line
+	5700 2800 5900 2800
+Wire Wire Line
+	5900 2800 5900 3350
+Wire Wire Line
+	5900 3350 4450 3350
+Wire Wire Line
+	4450 3350 4450 2800
+Connection ~ 4450 2800
+Wire Wire Line
+	6400 1100 6400 2000
+Wire Wire Line
+	6150 2000 7850 2000
+Wire Wire Line
+	4500 2600 4150 2600
+Wire Wire Line
+	4150 2600 4150 3650
+Wire Wire Line
+	4150 3650 6500 3650
+Wire Wire Line
+	6500 3650 6500 2600
+Wire Wire Line
+	6150 2600 7650 2600
+$Comp
+L R R36
+U 1 1 57D18B13
+P 6000 2600
+F 0 "R36" V 6080 2600 50  0000 C CNN
+F 1 "0R" V 6000 2600 50  0000 C CNN
+F 2 "" V 5930 2600 50  0000 C CNN
+F 3 "" H 6000 2600 50  0000 C CNN
+	1    6000 2600
+	0    1    1    0
+$EndComp
+Wire Wire Line
+	5850 2600 5700 2600
+Connection ~ 6500 2600
+$Comp
+L R R35
+U 1 1 57D18CB8
+P 6000 2000
+F 0 "R35" V 6080 2000 50  0000 C CNN
+F 1 "0R" V 6000 2000 50  0000 C CNN
+F 2 "" V 5930 2000 50  0000 C CNN
+F 3 "" H 6000 2000 50  0000 C CNN
+	1    6000 2000
+	0    1    1    0
+$EndComp
+Wire Wire Line
+	5850 2000 5700 2000
+Connection ~ 6400 2000
 $EndSCHEMATC

Commit message: Footprint atualizado
Parts:
- C4, C5: footprint (none) -> Capacitores:Cap_MKT_EPCOS_7,3x2,5
- IC1: footprint DIL16 -> Housings_DIP:DIP-16_W7.62mm_LongPads
- P4: footprint (none) -> Connect:Wafer_Vertical15x5.8x7RM2.5-5
- R29, R30: footprint (none) -> Resistors_ThroughHole:Resistor_Horizontal_RM15mm
- R35, R36: footprint (none) -> Resistors_SMD:R_1210_HandSoldering
Changed lines of the file:
@@
 F 0 "IC1" H 4700 3140 50  0000 L CNN
 F 1 "L293D" H 4700 1400 50  0000 L CNN
-F 2 "DIL16" H 5100 2300 50  0001 L CNN
+F 2 "Housings_DIP:DIP-16_W7.62mm_LongPads" H 5100 2300 50  0001 L CNN
 F 3 "DIP-16 STMicroelectronics" H 5100 2300 50  0001 L CNN
 F 4 "L293D" H 5100 2300 50  0001 L CNN "MP"
@@
 F 0 "P4" H 9800 3500 50  0000 C CNN
 F 1 "LOCK_CONNECTOR" V 9900 3200 50  0000 C CNN
-F 2 "" H 9800 3200 50  0000 C CNN
+F 2 "Connect:Wafer_Vertical15x5.8x7RM2.5-5" H 9800 3200 50  0001 C CNN
 F 3 "" H 9800 3200 50  0000 C CNN
 	1    9800 3200
@@
 F 0 "R29" V 8430 3000 50  0000 C CNN
 F 1 "R" V 8350 3000 50  0000 C CNN
-F 2 "" V 8280 3000 50  0000 C CNN
+F 2 "Resistors_ThroughHole:Resistor_Horizontal_RM15mm" V 8280 3000 50  0001 C CNN
 F 3 "" H 8350 3000 50  0000 C CNN
 F 4 "NOTA3" V 8250 3000 60  0000 C CNN "Nota"
@@
 F 0 "R30" V 8430 3400 50  0000 C CNN
 F 1 "R" V 8350 3400 50  0000 C CNN
-F 2 "" V 8280 3400 50  0000 C CNN
+F 2 "Resistors_ThroughHole:Resistor_Horizontal_RM15mm" V 8280 3400 50  0001 C CNN
 F 3 "" H 8350 3400 50  0000 C CNN
 F 4 "NOTA3" V 8250 3400 60  0000 C CNN "Nota"
@@
 F 0 "C5" H 6925 1600 50  0000 L CNN
 F 1 "100nF" H 6925 1400 50  0000 L CNN
-F 2 "" H 6938 1350 50  0000 C CNN
+F 2 "Capacitores:Cap_MKT_EPCOS_7,3x2,5" H 6938 1350 50  0001 C CNN
 F 3 "" H 6900 1500 50  0000 C CNN
 F 4 "NOTA2" H 7150 1500 60  0000 C CNN "Nota"
@@
 F 0 "C4" H 3525 2500 50  0000 L CNN
 F 1 "100nF" H 3525 2300 50  0000 L CNN
-F 2 "" H 3538 2250 50  0000 C CNN
+F 2 "Capacitores:Cap_MKT_EPCOS_7,3x2,5" H 3538 2250 50  0001 C CNN
 F 3 "" H 3500 2400 50  0000 C CNN
 F 4 "NOTA2" H 3250 2400 60  0000 C CNN "Nota"
@@
 F 0 "R36" V 6080 2600 50  0000 C CNN
 F 1 "0R" V 6000 2600 50  0000 C CNN
-F 2 "" V 5930 2600 50  0000 C CNN
+F 2 "Resistors_SMD:R_1210_HandSoldering" V 5930 2600 50  0001 C CNN
 F 3 "" H 6000 2600 50  0000 C CNN
 	1    6000 2600
@@
 F 0 "R35" V 6080 2000 50  0000 C CNN
 F 1 "0R" V 6000 2000 50  0000 C CNN
-F 2 "" V 5930 2000 50  0000 C CNN
+F 2 "Resistors_SMD:R_1210_HandSoldering" V 5930 2000 50  0001 C CNN
 F 3 "" H 6000 2000 50  0000 C CNN
 	1    6000 2000
