File: src/placa_microfone/placa_microfone.sch (KiCad schematic (older format))
At the start: 1 part

Commit message: Desenvolvida PCB para circuito mic_v2
Parts:
- added C1, C2, C3: 10u, Capacitors_ThroughHole:C_Radial_D5_L6_P2.5, symbol C
- added C4: 47n, Capacitors_ThroughHole:C_Disc_D3_P2.5, symbol C
- added C5: 100n, Capacitors_ThroughHole:C_Disc_D3_P2.5, symbol C
- added C6: 100u, Capacitors_ThroughHole:C_Radial_D5_L6_P2.5, symbol C
- added D1: 3V3 ZENER, Diodes_ThroughHole:Diode_DO-35_SOD27_Horizontal_RM10, symbol ZENER
- added R1: 10k, Resistors_ThroughHole:Resistor_Horizontal_RM7mm, symbol R
- added R2: 10R, Resistors_ThroughHole:Resistor_Horizontal_RM7mm, symbol R
- added U1: MIC_ELECTRET, Buzzers_Beepers:MagneticBuzzer_Kingstate_KCG0601, symbol MIC_ELECTRET
- added U2: LM386, Housings_DIP:DIP-8_W7.62mm_LongPads, symbol LM386
- P1: renamed from P?; footprint (none) -> Connect:Wafer_Vertical17.5x5.8x7RM2.5-6
Connections:
- net labels added: +5V
- net labels removed: +12V
- wire segments 5 -> 40
- no-connect marks 0 -> 3
